File: v7_RK3588_PCB/RK3588.kicad_sch (KiCad schematic)
At the start: 0 parts

Commit message: add symbols
Parts:
- added U2001: ~, RK3588:FCBGA-1088_L23.0-W23.0-P0.65-TL_RK3588, symbol RK3588:RK3588_C5156490

Commit message: add ESP32 schematic
Parts:
- added C2001, C2007: 100nF/10V, symbol Device:C
- added C2002: 10n/25V, symbol Device:C
- added C2003, C2004: 9pF/50V, symbol Device:C
- added C2005: 1nF/50V, symbol Device:C
- added C2006: 10uF/10V, symbol Device:C
- added C2008, C2011: 100nF/6.3V, symbol Device:C
- added C2009: 1n/50V, symbol Device:C
- added C2010: 100n/16V, symbol Device:C
- added D2001, D2002: PJE5UFN10A-AU_R1_000A1, symbol PJE5UFN10A-AU_R1_000A1:PJE5UFN10A-AU_R1_000A1
- added D2003, D2004: D_TVS, ESD5451N2:DFN1006-2L_TWS, symbol Device:D_TVS
- added J2001: Micro_SD_Card_Det1, symbol Connector:Micro_SD_Card_Det1
- added J2002: Conn_01x04_Pin, symbol Connector:Conn_01x04_Pin
- added R2001, R2009, R2010, R2011, R2012, R2013, R2014: 22, symbol Device:R
- added R2002, R2003, R2015: 10k, symbol Device:R
- added R2004: 0, symbol Device:R
- added R2005: 510k, symbol Device:R
- added R2006: 100k, symbol Device:R
- added R2007: 20k, symbol Device:R
- added R2008, R2016, R2017: 100, symbol Device:R
- added X2001: TSX-3225 24.0000MF20G-AC0, TSX-3225_footprints:CRYSTAL_TSX-3225_TSX-3225 24.0000MF20G-AC0_EPS, symbol CRYSTAL_TSX_3225_24_0000MF20G_AC0:TSX-3225_24.0000MF20G-AC0
Connections:
- net NPOR_u: now reaches U2001.M31 (NPOR_u)
- net NPOR_u: now also C2001.1, R2004.1
- net at U2001.AL16 (SARADC_IN1): now also C2009.1, R2015.2
- net at U2001.AM16 (SARADC_IN0_BOOT): now also C2005.1, R2006.2, R2007.1
- net SDMMC0_CLK: now reaches U2001.AE1 (SDMMC_CLK/PDM1_CLK0_M0/TEST_CLKOUT_M0/MCU_JTAG_TMS_M0/CAN0_RX_M1/UART5_TX_M0/GPIO4_D5_d)
- net SDMMC0_CLK: now also R2011.2
- net SDMMC0_CMD: now reaches U2001.AE2 (SDMMC_CMD/PDM1_CLK1_M0/MCU_JTAG_TCK_M0/CAN0_TX_M1/UART5_RX_M0/PWM7_IR_M1/GPIO4_D4_u)
- net SDMMC0_CMD: now also R2012.2
- net SDMMC0_D3: now reaches U2001.AF1 (SDMMC_D3/PDM1_SDI0_M0/JTAG_TMS_M0/I2C8_SDA_M0/UART5_RTSN_M0/PWM10_M1/GPIO4_D3_u)
- net SDMMC0_D3: now also R2013.2
- net SDMMC0_D2: now reaches U2001.AF2 (SDMMC_D2/PDM1_SDI1_M0/JTAG_TCK_M0/I2C8_SCL_M0/UART5_CTSN_M0/GPIO4_D2_u)
- net SDMMC0_D2: now also R2014.2
- net XOUT24M: now reaches U2001.T34 (XOUT_24M)
- net XOUT24M: now also R2001.2, R2005.1
- net  VCCIO_SD_S0: now reaches U2001.Y7 (VCCIO2)
- net  VCCIO_SD_S0: now also C2011.1
- net UART2_TX_M0: now reaches U2001.P30 (I2S1_SDI0_M1/GPU_AVS/UART0_TX_M0/I2C4_SCL_M2/DP1_HPDIN_M1/PWM4_M0/PCIE30X1_0_PERSTN_M0/GPIO0_C5_u)
- net UART2_TX_M0: now also R2016.1
- net SDMMC0_DET_L: now reaches U2001.P31 (SDMMC_DET/GPIO0_A4_u)
- net SDMMC0_DET_L: now also R2008.2
- net UART2_RX_M0: now reaches U2001.R29 (I2S1_SCLK_TX_M1/JTAG_TMS_M2/I2C1_SDA_M0/UART2_RX_M0/PCIE30X1_1_WAKEN_M0/GPIO0_B6_d)
- net UART2_RX_M0: now also R2017.1
- net XIN24M: now reaches U2001.R34 (XIN_24M)
- net XIN24M: now also C2003.1, R2005.2, X2001.3
- net  VCC_1V8_S0: now reaches U2001.AA7 (VCCIO2_1V8)
- net  VCC_1V8_S0: now also C2008.1
- net SDMMC0_D1: now reaches U2001.AD1 (SDMMC_D1/PDM1_SDI2_M0/JTAG_TMS_M1/I2C3_SDA_M4/UART2_RX_M1/PWM9_M1/GPIO4_D1_u)
- net SDMMC0_D1: now also R2009.2
- net SDMMC0_D0: now reaches U2001.AD2 (SDMMC_D0/PDM1_SDI3_M0/JTAG_TCK_M1/I2C3_SCL_M4/UART2_TX_M1/PWM8_M1/GPIO4_D0_u)
- net SDMMC0_D0: now also R2010.2
- new net: D2001.4 (I/O_3), J2001.3 (CMD), R2012.1
- new net: D2004.2 (A2), J2002.2 (Pin_2), R2016.2
- new net: D2003.2 (A2), J2002.3 (Pin_3), R2017.2
- new net: C2004.1, R2001.1, X2001.1
- new net: D2001.2 (I/O_2), J2001.2 (DAT3/CD), R2013.1
- new net: D2002.1 (I/O_1), J2001.9 (DET), R2008.1
- new net: D2002.2 (I/O_2), J2001.8 (DAT1), R2009.1
- new net: D2002.4 (I/O_3), J2001.7 (DAT0), R2010.1
- new net: D2002.5 (I/O_4), J2001.5 (CLK), R2011.1
- new net: D2001.1 (I/O_1), J2001.1 (DAT2), R2014.1
- new net GND: C2001.2, C2002.2, C2003.2, C2004.2, C2005.2, C2006.2, C2007.2, C2008.2, C2009.2, C2010.1, C2011.2, D2001.3 (GND_1), D2001.8 (GND_2), D2002.3 (GND_1), D2002.8 (GND_2), D2003.1 (A1), D2004.1 (A1), J2001.10 (SHIELD), J2001.6 (VSS), J2002.4 (Pin_4), R2007.2, X2001.2, X2001.4
- new net PMIC_INT_L: R2002.2
- new net RESET_L: C2002.1, R2003.2
- new net TSADC_SHUT_H: R2004.2
- new net VCC3V3_SD: C2006.1, C2007.1, J2001.4 (VDD)
- new net VCCA_1V8_S0: R2006.1, R2015.1
- new net VCC_1V8_S3: R2002.1, R2003.1
- new net VCC_3V3_S3: C2010.2, J2002.1 (Pin_1)
- no-connect marks 0 -> 9
Other:
- note added: "2.1.1 Clock Circuit"
- note added: "2.1.2 Reset/watchdog/TSADC Circuit"
- note added: "2.1.4 System Boot Sequence via SDMMC0 Card"
- note added: "2.1.6 UART Debug"
- note added: "TODO: cap calc design guide pg 21"
- note added: "TODO: check if all resistors"
- note added: "config. for SD card boot"
- note added: "place close to chip"
- note added: "place close to uSD"
