File: v7_RK3588_PCB/ESP32.kicad_sch (KiCad schematic)
At the start: 0 parts

Commit message: add ESP32 schematic
Parts:
- added C? (x3): 0.1uF, symbol Device:C
- added C? (x2): 10pF, symbol Device:C
- added C? (x3): 1uF, symbol Device:C
- added C? (x2): 10uF, symbol Device:C
- added C? (x2): C, symbol Device:C
- added D?: LED, LED_SMD:LED_0805_2012Metric_Pad1.15x1.40mm_HandSolder, symbol Device:LED
- added J?: 2337019-1, CONN_2337019-1, symbol CONN_2337019-1:2337019-1
- added J?: Conn_01x05_Pin, symbol Connector:Conn_01x05_Pin
- added J?: Micro_SD_Card_Det1, symbol Connector:Micro_SD_Card_Det1
- added J?: Conn_01x04_Pin, symbol Connector:Conn_01x04_Pin
- added J?: Conn_01x02_Pin, symbol Connector:Conn_01x02_Pin
- added L?: 2nH, symbol Device:L
- added L?: L, symbol Device:L
- added L?: 24nH, symbol Device:L
- added R? (x6): 10K, symbol Device:R
- added R? (x7): 22, symbol Device:R
- added R?: 10k, symbol Device:R
- added R?: 0, symbol Device:R
- added R?: 499, symbol Device:R
- added R?: 270, symbol Device:R
- added R?: 4.7k, symbol Device:R
- added U?: ESP32-C6FH4, ESP32-C6FH4:QFN50P500X500X90-33N, symbol ESP32-C6FH4:ESP32-C6FH4
- added X?: FW400WFMR1, Crystal_FW400WFMR1:Crystal_FW400_DIO, symbol FW400WFMR1:FW400WFMR1
Connections:
- new net: J?.1 (DAT2), R?.1, R?.1
- new net: J?.5 (CLK), R?.1
- new net: J?.2 (DAT3/CD), R?.1, R?.1
- new net: C?.1, L?.1, U?.2 (VDDA3P3), U?.3 (VDDA3P3__1)
- new net: C?.2, R?.2, U?.4 (CHIP_PU)
- new net: D?.2 (A), R?.2
- new net: J?.9 (DET), R?.1, R?.1
- new net: R?.2, U?.15 (GPIO9)
- new net: R?.1, U?.21 (U0TXD/GPIO16)
- new net: C?.2, U?.30 (XTAL_N), X?.3
- new net: L?.2, U?.31 (XTAL_P)
- new net: C?.2, L?.1, X?.1
- new net: J?.3 (CMD), R?.1, R?.1
- new net: J?.7 (DAT0), R?.1, R?.1
- new net: J?.8 (DAT1), R?.1, R?.1
- new net ESP_I2C1_SCL: U?.6 (GPIO0/XTAL_32K_P)
- new net ESP_I2C1_SDA: U?.7 (GPIO1/XTAL_32K_N)
- new net GND: C?.1, C?.1, C?.1, C?.2, C?.2, C?.2, C?.2, C?.2, C?.2, C?.2, C?.2, C?.2, D?.1 (K), J?.10 (SHIELD), J?.2, J?.3, J?.4 (Pin_4), J?.6 (VSS), U?.33 (GND), X?.2, X?.4
- new net GPIO12: J?.1 (Pin_1), U?.16 (USB_D-/GPIO12)
- new net GPIO13: J?.2 (Pin_2), U?.17 (USB_D+/GPIO13)
- new net GPIO2: R?.1, U?.8 (GPIO2)
- new net GPIO4: J?.1 (Pin_1), U?.10 (GPIO4/MTMS)
- new net GPIO5: J?.2 (Pin_2), U?.11 (GPIO5/MTDI)
- new net GPIO6: J?.3 (Pin_3), U?.12 (GPIO6/MTCK)
- new net GPIO7: J?.4 (Pin_4), U?.13 (GPIO7/MTDO)
- new net GPIO8: J?.5 (Pin_5), U?.14 (GPIO8)
- new net LNA_IN: C?.1, L?.1, U?.1 (ANT)
- new net PMIC_PWRON: U?.18 (GPIO14)
- new net RF_ANT: C?.1, J?.1, L?.2
- new net SDMMC0_CLK: R?.2, U?.24 (SDIO_CLK/GPIO19)
- new net SDMMC0_CMD: R?.2, U?.23 (SDIO_CMD/GPIO18)
- new net SDMMC0_D0: R?.2, U?.25 (SDIO_DATA0/GPIO20)
- new net SDMMC0_D1: R?.2, U?.26 (SDIO_DATA1/GPIO21)
- new net SDMMC0_D2: R?.2, U?.27 (SDIO_DATA2/GPIO22)
- new net SDMMC0_D3: R?.2, U?.28 (SDIO_DATA3/GPIO23)
- new net SDMMC0_DET_L: R?.2, U?.9 (GPIO3)
- new net UART0_RXD: J?.2 (Pin_2), U?.22 (U0RXD/GPIO17)
- new net UART0_TXD: J?.1 (Pin_1), R?.2
- new net VCC3V3_SYS: J?.4 (VDD), R?.2, R?.2, R?.2, R?.2, R?.2, R?.2
- new net VCC_3V3: R?.1
- new net VDD3V3_ESP: C?.1, C?.1, C?.1, C?.1, C?.1, C?.1, J?.3 (Pin_3), L?.2, R?.1, R?.1, R?.2, U?.20 (VDDPST2), U?.29 (VDDA1), U?.32 (VDDA2), U?.5 (VDDPST1)
- no-connect marks 0 -> 1
Other:
- note added: "Checked: Saul"
- note added: "UART connector for firmware download"

Commit message: add power sequencing
Parts:
- J4001: renamed from J?; footprint CONN_2337019-1 -> (none)
- gave numbers to parts that had none: 40
