File: v7_RK3588_PCB/Ethernet.kicad_sch (KiCad schematic)
At the start: 0 parts

Commit message: add ethernet schematic
Parts:
- added C7001, C7004, C7009, C7010, C7011: 4.7uF/6.3V/10%/X7R, symbol Device:C
- added C7002, C7005, C7006, C7007, C7008, C7012: 0.1uF/6.3V/10%/X7R, symbol Device:C
- added C7003: 10uF/6.3V/10%/X7R, symbol Device:C
- added C7013: 10nF/100V/1%/X7R, symbol Device:C
- added C7014, C7018, C7027: 0.1uF/100V/1%/X7R, symbol Device:C
- added C7015: 47uF/63V/1%/X7R, symbol Device:C_Polarized_US
- added C7016, C7017, C7028, C7030: 1uF/100V/1%/X7R, symbol Device:C
- added C7019, C7020, C7021: 47uF/25V/1%/X7R, symbol Device:C
- added C7022, C7023: 330uF/25V/1%/X7R, symbol Device:C_Polarized_US
- added C7024, C7037: 1uF/25V/1%/X7R, symbol Device:C
- added C7025: 1.2nF/25V/1%/X7R, symbol Device:C
- added C7026: 1nF/100V/1%/X7R, symbol Device:C
- added C7029: 22uF/100V/1%/X7R, symbol Device:C_Polarized_US
- added C7031, C7032: 0.47uF/100V/1%/X7R, symbol Device:C
- added C7033: 2.2nF/100V/1%/X7R, symbol Device:C
- added C7034: 3.3nF/25V/1%/X7R, symbol Device:C
- added C7035: 27nF/25V/1%/X7R, symbol Device:C
- added C7036: 10nF/25V/1%/X7R, symbol Device:C
- added CR7001: B1100-13-F, SMA_DIO, symbol B1100_13_F:B1100-13-F
- added D7001, D7005: SMAJ58A, Diode_SMD:D_SMA, symbol Diode:SMAJ58A
- added D7002, D7003: BAV20WS, symbol BAV20WS:Diode
- added D7004, D7006: BAV99, Package_TO_SOT_SMD:SOT-23, symbol Diode:BAV99
- added FB? (x2): 500@100M/3A, symbol Device:FerriteBead
- added FB?: 600@100M/250mA, symbol Device:FerriteBead
- added J7001: ARJ-139, symbol arj139:ARJ-139
- added L7001: 3.3uH/3A, symbol Device:L_Iron
- added L7002: 0.33uH/5A, symbol Device:L_Iron
- added Q?: SIR464DP, Package_SO:Vishay_PowerPAK_1212-8_Single, symbol Simulation_SPICE:NMOS
- added Q?: SI7898DP-T1-E3, MOSFET_50DP-T1-E3_VIS, symbol SI7898DP:SI7898DP-T1-E3
- added Q?: LP0701, symbol Simulation_SPICE:PMOS
- added Q?: MMBT3906, Package_TO_SOT_SMD:SOT-23, symbol Transistor_BJT:MMBT3906
- added R7001: 220/5%, symbol Device:R
- added R7002: 200/5%, symbol Device:R
- added R7003, R7004: 1K/5%, symbol Device:R
- added R7005: 1.5K/1%, symbol Device:R
- added R7006, R7007, R7008, R7009, R7010, R7011, R7012, R7013, R7014, R7015, R7016, R7017, R7018, R7020: 22/1%, symbol Device:R
- added R7019, R7033, R7036: 10K/1%, symbol Device:R
- added R7021: 12.1K/1%, symbol Device:R
- added R7022: 39k/0.1W, symbol Device:R
- added R7023: 24.9K/1%, symbol Device:R
- added R7024, R7025, R7030: 10/1%, symbol Device:R
- added R7026: 63.4/0.1W/1%, symbol Device:R
- added R7027: 38.3K/1%, symbol Device:R
- added R7028, R7029: 69.8K/1%, symbol Device:R
- added R7031: 1K/1%, symbol Device:R
- added R7032: 0.18/0.5W, symbol Device:R
- added R7034: 49.9/1%, symbol Device:R
- added R7035: 449/1%, symbol Device:R
- added R7037: 2K/1%, symbol Device:R
- added R7038: 604/1%, symbol Device:R
- added R7039: 41.2K/1%, symbol Device:R
- added R7040: 13.7K/1%, symbol Device:R
- added T?: PA0184NL, Transformer_SMD:Pulse_PA2007NL, symbol Transformer:PA0184NL
- added T?: POE300F-50LD, POE300F30LD, symbol POE300F-50LD:POE300F-50LD
- added TP? (x12): TestPoint, symbol Connector:TestPoint
- added U7001: KSZ9031RNXCA, Package_DFN_QFN:QFN-48-1EP_7x7mm_P0.5mm_EP5.15x5.15mm, symbol Interface_Ethernet:KSZ9031RNXCA
- added U7002, U7004: CDBHM1100L-HF, CDBHM1100L-HF_CIP, symbol CBDHM1100L-HF:CDBHM1100L-HF
- added U7003: TPS23754PWP, PWP20_3P4X2P4, symbol TPS23754PWP:TPS23754PWP
- added U7005: TCMT1107, Package_SO:SOP-4_4.4x2.6mm_P1.27mm, symbol Isolator:TCMT1107
- added U7006: TLV431ASN1T1G, SOT-23_ONS, symbol TLV431ASN1T1G:TLV431ASN1T1G
Connections:
- new net: D7006.2 (A), R7034.1, R7036.1, R7038.1, R7039.1, TP?.1
- new net: C7036.1, C7037.1, D7006.1 (K), D7006.3 (K), R7036.2, U7005.2, U7006.2 (CATHODE)
- new net: C7035.1, R7035.2
- new net: C7034.2, C7035.2, R7037.2, TP?.1, U7003.1 (CTL), U7005.4
- new net: C7019.1, C7020.1, C7021.1, C7022.1, L7002.1, T?.7 (SEC_1), T?.8 (SEC_2), T?.9 (SEC_3)
- new net: R7009.2, U7001.20 (TXD1)
- new net: R7028.1, U7003.18 (BLNK)
- new net: C7013.2, C7014.1, C7015.1, CR7001.1, L7001.1, U7003.11 (VDD1)
- new net: C7013.1, C7027.1, CR7001.2, D7001.1 (A1), FB?.2, R7023.1, TP?.1, U7003.12 (VDD)
- new net: C7016.1, C7017.1, C7018.1, L7001.2, R7022.1, T?.1 (PRI_1), T?.2 (PRI_2)
- new net: C7018.2, D7002.2 (C), R7022.2
- new net: C7027.2, D7001.2 (A2), D7005.2 (A2), FB?.2, R7026.2, TP?.1, U7003.10 (VSS), U7003.21 (EPAD)
- new net: R7023.2, U7003.13 (DEN)
- new net: R7026.1, U7003.15 (CLS)
- new net: R7027.1, U7003.16 (DT)
- new net: R7029.1, U7003.19 (FRS)
- new net: C7030.1, C7034.1, R7035.1, R7037.1, TP?.1, U7003.2 (VS)
- new net: R7031.1, TP?.1, U7003.3 (CS)
- new net: R7030.1, TP?.1, U7003.5 (GATE)
- new net: C7028.1, C7029.1, D7003.2 (C), TP?.1, U7003.6 (VC)
- new net: C7032.1, U7003.7 (GAT2)
- new net: C7006.2, C7009.2, FB?.2, U7001.14 (DVDDL), U7001.18 (DVDDL), U7001.23 (DVDDL), U7001.26 (DVDDL), U7001.30 (DVDDL), U7001.39 (DVDDL)
- new net: R7021.1, U7001.48 (ISET)
- new net: C7031.1, T?.5
- new net: C7031.2, D7004.3 (K), Q?.1 (B), R7033.1
- new net: C7032.2, T?.1
- new net: C7025.2, R7024.1
- new net: D7002.1 (A), Q?.5 (D), Q?.6 (D), Q?.7 (D), Q?.8 (D), T?.3 (PRI_3), T?.4 (PRI_4), TP?.1
- new net: R7017.2, U7001.27 (RXD3/MODE3)
- new net: R7007.2, U7001.25 (TX_EN)
- new net: R7014.2, U7001.32 (RXD0/MODE0)
- new net: C7025.1, Q?.1 (D), T?.10 (SEC_4), T?.11 (SEC_5), T?.12 (SEC_6)
- new net: D7004.2 (A), Q?.2 (E), Q?.2 (G)
- new net: Q?.1 (S), Q?.2 (S), Q?.3 (S), R7031.2, R7032.1
- new net: C7026.2, FB?.1, U7002.2, U7004.2
- new net: C7036.2, R7039.2, R7040.1, U7006.1 (REFERENCE)
- new net: C7007.2, C7008.2, C7010.2, C7011.2, C7012.1, FB?.1, Q?.1 (D), U7001.4 (AVDDL), U7001.44 (AVDDL_PLL), U7001.9 (AVDDL)
- new net: R7011.2, U7001.22 (TXD3)
- new net: C7026.1, FB?.1, U7002.1, U7004.1
- new net: Q?.4 (G), R7030.2
- new net: R7008.2, U7001.19 (TXD0)
- new net: R7010.2, U7001.21 (TXD2)
- new net: R7012.2, U7001.24 (GTX_CLK)
- new net: R7016.2, U7001.28 (RXD2/MODE2)
- new net: R7015.2, U7001.31 (RXD1/MODE1)
- new net: R7013.2, U7001.33 (RX_DV/CLK125_EN)
- new net: R7018.2, U7001.35 (RX_CLK/PHYAD2)
- new net: R7006.2, U7001.36 (MDC)
- new net: Q?.2 (G), U7001.43 (LDO_O)
- new net: R7020.1, U7001.46 (XI)
- new net: R7025.2, T?.6 (AUX_2)
- new net: R7038.2, U7005.1
- new net: J7001.17 (CATHODE_Y), R7001.2
- new net: J7001.20 (ANODE_G/CATHODE_O), R7002.2
- new net: D7003.1 (A), R7025.1
- new net 100M_LED_LOW: J7001.18 (ANODE_Y), R7004.2, U7001.17 (LED1/PHAD0/PME_N1)
- new net 1G_LED_LOW: J7001.19 (ANODE_O/CATHODE_G), R7003.1, U7001.15 (LED2/PHYAD1)
- new net 5V0_OUT_ETH: C7023.1, C7024.1, L7002.2, R7034.2, TP?.1
- new net CT_0: J7001.1 (CT), U7002.3
- new net CT_1: J7001.6 (CT), U7002.4
- new net CT_2: J7001.7 (CT), U7004.3
- new net CT_3: J7001.12 (CT), U7004.4
- new net ETHERNET_RESET_GPIO: R7019.1, U7001.42 (RESET_N)
- new net ETHO_REFCLKO_25M: R7020.2
- new net GMAC1_MDC: R7006.1
- new net GMAC1_MDIO: R7005.2, U7001.37 (MDIO)
- new net GMAC1_RXCLK: R7018.1
- new net GMAC1_RXD0: R7014.1
- new net GMAC1_RXD1: R7015.1
- new net GMAC1_RXD2: R7016.1
- new net GMAC1_RXD3: R7017.1
- new net GMAC1_RXDV_CRS: R7013.1
- new net GMAC1_TXCLK: R7012.1
- new net GMAC1_TXD0: R7008.1
- new net GMAC1_TXD1: R7009.1
- new net GMAC1_TXD2: R7010.1
- new net GMAC1_TXD3: R7011.1
- new net GMAC1_TXEN: R7007.1
- new net GND: C7001.1, C7002.1, C7003.1, C7004.1, C7005.1, C7006.1, C7007.1, C7008.1, C7009.1, C7010.1, C7011.1, C7012.2, C7019.2, C7020.2, C7021.2, C7022.2, C7023.2, C7024.2, C7033.2, C7037.2, D7004.1 (K), Q?.3 (C), Q?.3 (S), R7003.2, R7004.1, R7021.2, R7024.2, R7033.2, R7040.2, T?.4, U7001.29 (VSS), U7001.49 (PAD_GND), U7003.17 (APD), U7006.3 (ANODE)
- new net GND_RTN: C7014.2, C7015.2, C7016.2, C7017.2, C7028.2, C7029.2, C7030.2, C7033.1, D7005.1 (A1), R7027.2, R7028.2, R7029.2, R7032.2, T?.5 (AUX_1), T?.8, TP?.1, TP?.1, U7003.4 (COM), U7003.8 (ARTN), U7003.9 (RTN), U7005.3
- new net T2P: U7003.20 (T2P)
- new net TXRXM_0: J7001.10 (TRD0-), U7001.3 (TXRXM_A)
- new net TXRXM_1: J7001.5 (TRD1-), U7001.6 (TXRXM_B)
- new net TXRXM_2: J7001.2 (TRD2-), U7001.8 (TXRXM_C)
- new net TXRXM_3: J7001.9 (TRD3-), U7001.11 (TXRXM_D)
- new net TXRXP_0: J7001.11 (TRD0+), U7001.2 (TXRXP_A)
- new net TXRXP_1: J7001.4 (TRD1+), U7001.5 (TXRXP_B)
- new net TXRXP_2: J7001.3 (TRD2+), U7001.7 (TXRXP_C)
- new net TXRXP_3: J7001.8 (TRD3+), U7001.10 (TXRXP_D)
- new net VCC_1V8: C7003.2, C7004.2, C7005.2, R7005.1, R7019.2, U7001.16 (DVDDH), U7001.34 (DVDDH), U7001.40 (DVDDH)
- new net VCC_3V3: C7001.2, C7002.2, Q?.3 (S), R7001.1, R7002.1, U7001.1 (AVDDH), U7001.12 (AVDDH)
- no-connect marks 0 -> 9
Other:
- note added: "Checked: Tamar"
- note added: "Clock from SoC"
- note added: "Ethernet PHY"
- note added: "Grounds Isolation"
- note added: "Place decoupling caps as close as possible to Ethernet PHY"
- note added: "Place resistors closest to the side indicated."
- note added: "PoE Interface"
- note added: "RJ45 + Magnetics Ethernet Jack"
- note added: "flyback transformer"

Commit message: add power sequencing
Parts:
- CR7001: footprint SMA_DIO -> (none)
- Q7003: renamed from Q?; footprint MOSFET_50DP-T1-E3_VIS -> (none)
- T7001: renamed from T?; footprint POE300F30LD -> (none)
- U7002, U7004: footprint CDBHM1100L-HF_CIP -> (none)
- U7003: footprint PWP20_3P4X2P4 -> (none)
- U7006: footprint SOT-23_ONS -> (none)
- gave numbers to parts that had none: 19
Changed lines of the file:
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@@
 		(dnp no)
 		(fields_autoplaced yes)
-		(property "Reference" "TP?"
+		(property "Reference" "TP7012"
 			(at 284.48 344.6779 0)
 			(effects
@@
 			(project "v7_RK3588_PCB"
 				(path "/1d5a1342-f497-4807-8bdb-ea718133b0ad/fb1254ad-a22e-4d7b-81d8-e9d32dd5de93"
-					(reference "TP?")
+					(reference "TP7012")
 					(unit 1)
 				)
@@
 			)
 		)
-		(property "Footprint" "SMA_DIO"
+		(property "Footprint" ""
 			(at 144.78 227.33 0)
 			(effects
@@
 			)
 		)
-		(property "Footprint" "PWP20_3P4X2P4"
+		(property "Footprint" ""
 			(at 223.52 265.43 0)
 			(effects
@@
 		(dnp no)
 		(fields_autoplaced yes)
-		(property "Reference" "TP?"
+		(property "Reference" "TP7001"
 			(at 125.73 222.7579 0)
 			(effects
@@
 			(project "v7_RK3588_PCB"
 				(path "/1d5a1342-f497-4807-8bdb-ea718133b0ad/fb1254ad-a22e-4d7b-81d8-e9d32dd5de93"
-					(reference "TP?")
+					(reference "TP7001")
 					(unit 1)
 				)
@@
 		(on_board yes)
 		(dnp no)
-		(property "Reference" "T?"
+		(property "Reference" "T7002"
 			(at 339.09 306.07 0)
 			(effects
@@
 			(project "v7_RK3588_PCB"
 				(path "/1d5a1342-f497-4807-8bdb-ea718133b0ad/fb1254ad-a22e-4d7b-81d8-e9d32dd5de93"
-					(reference "T?")
+					(reference "T7002")
 					(unit 1)
 				)
@@
 		(dnp no)
 		(fields_autoplaced yes)
-		(property "Reference" "TP?"
+		(property "Reference" "TP7004"
 			(at 328.93 255.2699 90)
 			(effects
@@
 			(project "v7_RK3588_PCB"
 				(path "/1d5a1342-f497-4807-8bdb-ea718133b0ad/fb1254ad-a22e-4d7b-81d8-e9d32dd5de93"
-					(reference "TP?")
+					(reference "TP7004")
 					(unit 1)
 				)
@@
 		(on_board yes)
 		(dnp no)
-		(property "Reference" "TP?"
+		(property "Reference" "TP7006"
 			(at 221.488 269.24 90)
 			(effects
@@
 			(project "v7_RK3588_PCB"
 				(path "/1d5a1342-f497-4807-8bdb-ea718133b0ad/fb1254ad-a22e-4d7b-81d8-e9d32dd5de93"
-					(reference "TP?")
+					(reference "TP7006")
 					(unit 1)
 				)
@@
 		(on_board yes)
 		(dnp no)
-		(property "Reference" "Q?"
+		(property "Reference" "Q7002"
 			(at 411.734 262.89 90)
 			(effects
@@
 			(project "v7_RK3588_PCB"
 				(path "/1d5a1342-f497-4807-8bdb-ea718133b0ad/fb1254ad-a22e-4d7b-81d8-e9d32dd5de93"
-					(reference "Q?")
+					(reference "Q7002")
 					(unit 1)
 				)
@@
 		(dnp no)
 		(fields_autoplaced yes)
-		(property "Reference" "TP?"
+		(property "Reference" "TP7005"
 			(at 279.4 268.4779 0)
 			(effects
@@
 			(project "v7_RK3588_PCB"
 				(path "/1d5a1342-f497-4807-8bdb-ea718133b0ad/fb1254ad-a22e-4d7b-81d8-e9d32dd5de93"
-					(reference "TP?")
+					(reference "TP7005")
 					(unit 1)
 				)
@@
 		(on_board yes)
 		(dnp no)
-		(property "Reference" "FB?"
+		(property "Reference" "FB7003"
 			(at 111.76 280.416 90)
 			(effects
@@
 			(project "v7_RK3588_PCB"
 				(path "/1d5a1342-f497-4807-8bdb-ea718133b0ad/fb1254ad-a22e-4d7b-81d8-e9d32dd5de93"
-					(reference "FB?")
+					(reference "FB7003")
 					(unit 1)
 				)
@@
 		(dnp no)
 		(fields_autoplaced yes)
-		(property "Reference" "TP?"
+		(property "Reference" "TP7003"
 			(at 269.24 254.7619 0)
 			(effects
@@
 			(project "v7_RK3588_PCB"
 				(path "/1d5a1342-f497-4807-8bdb-ea718133b0ad/fb1254ad-a22e-4d7b-81d8-e9d32dd5de93"
-					(reference "TP?")
+					(reference "TP7003")
 					(unit 1)
 				)
@@
 		(dnp no)
 		(fields_autoplaced yes)
-		(property "Reference" "TP?"
+		(property "Reference" "TP7007"
 			(at 279.4 280.1619 0)
 			(effects
@@
 			(project "v7_RK3588_PCB"
 				(path "/1d5a1342-f497-4807-8bdb-ea718133b0ad/fb1254ad-a22e-4d7b-81d8-e9d32dd5de93"
-					(reference "TP?")
+					(reference "TP7007")
 					(unit 1)
 				)
@@
 			)
 		)
-		(property "Footprint" "CDBHM1100L-HF_CIP"
+		(property "Footprint" ""
 			(at 49.53 236.22 0)
 			(effects
@@
 		(dnp no)
 		(fields_autoplaced yes)
-		(property "Reference" "Q?"
+		(property "Reference" "Q7003"
 			(at 328.93 266.6999 0)
 			(effects
@@
 			)
 		)
-		(property "Footprint" "MOSFET_50DP-T1-E3_VIS"
+		(property "Footprint" ""
 			(at 314.96 270.51 0)
 			(effects
@@
 			(project "v7_RK3588_PCB"
 				(path "/1d5a1342-f497-4807-8bdb-ea718133b0ad/fb1254ad-a22e-4d7b-81d8-e9d32dd5de93"
-					(reference "Q?")
+					(reference "Q7003")
 					(unit 1)
 				)
@@
 		(dnp no)
 		(fields_autoplaced yes)
-		(property "Reference" "T?"
+		(property "Reference" "T7001"
 			(at 355.6 223.52 0)
 			(effects
@@
 			)
 		)
-		(property "Footprint" "POE300F30LD"
+		(property "Footprint" ""
 			(at 367.03 326.06 0)
 			(effects
@@
 			(project "v7_RK3588_PCB"
 				(path "/1d5a1342-f497-4807-8bdb-ea718133b0ad/fb1254ad-a22e-4d7b-81d8-e9d32dd5de93"
-					(reference "T?")
+					(reference "T7001")
 					(unit 1)
 				)
@@
 			)
 		)
-		(property "Footprint" "SOT-23_ONS"
+		(property "Footprint" ""
 			(at 435.61 372.11 0)
 			(effects
@@
 		(dnp no)
 		(fields_autoplaced yes)
-		(property "Reference" "TP?"
+		(property "Reference" "TP7010"
 			(at 323.85 324.3579 0)
 			(effects
@@
 			(project "v7_RK3588_PCB"
 				(path "/1d5a1342-f497-4807-8bdb-ea718133b0ad/fb1254ad-a22e-4d7b-81d8-e9d32dd5de93"
-					(reference "TP?")
+					(reference "TP7010")
 					(unit 1)
 				)
@@
 		(on_board yes)
 		(dnp no)
-		(property "Reference" "FB?"
+		(property "Reference" "FB7001"
 			(at 276.098 92.964 0)
 			(effects
@@
 			(project "v7_RK3588_PCB"
 				(path "/1d5a1342-f497-4807-8bdb-ea718133b0ad/fb1254ad-a22e-4d7b-81d8-e9d32dd5de93"
-					(reference "FB?")
+					(reference "FB7001")
 					(unit 1)
 				)
@@
 		(dnp no)
 		(fields_autoplaced yes)
-		(property "Reference" "Q?"
+		(property "Reference" "Q7001"
 			(at 266.7 107.9499 0)
 			(effects
@@
 			(project "v7_RK3588_PCB"
 				(path "/1d5a1342-f497-4807-8bdb-ea718133b0ad/fb1254ad-a22e-4d7b-81d8-e9d32dd5de93"
-					(reference "Q?")
+					(reference "Q7001")
 					(unit 1)
 				)
@@
 			)
 		)
-		(property "Footprint" "CDBHM1100L-HF_CIP"
+		(property "Footprint" ""
 			(at 49.53 270.51 0)
 			(effects
@@
 		(on_board yes)
 		(dnp no)
-		(property "Reference" "FB?"
+		(property "Reference" "FB7002"
 			(at 111.76 222.504 90)
 			(effects
@@
 			(project "v7_RK3588_PCB"
 				(path "/1d5a1342-f497-4807-8bdb-ea718133b0ad/fb1254ad-a22e-4d7b-81d8-e9d32dd5de93"
-					(reference "FB?")
+					(reference "FB7002")
 					(unit 1)
 				)
@@
 		(dnp no)
 		(fields_autoplaced yes)
-		(property "Reference" "TP?"
+		(property "Reference" "TP7008"
 			(at 171.45 286.5119 0)
 			(effects
@@
 			(project "v7_RK3588_PCB"
 				(path "/1d5a1342-f497-4807-8bdb-ea718133b0ad/fb1254ad-a22e-4d7b-81d8-e9d32dd5de93"
-					(reference "TP?")
+					(reference "TP7008")
 					(unit 1)
 				)
@@
 		(dnp no)
 		(fields_autoplaced yes)
-		(property "Reference" "TP?"
+		(property "Reference" "TP7002"
 			(at 488.95 222.7579 0)
 			(effects
@@
 			(project "v7_RK3588_PCB"
 				(path "/1d5a1342-f497-4807-8bdb-ea718133b0ad/fb1254ad-a22e-4d7b-81d8-e9d32dd5de93"
-					(reference "TP?")
+					(reference "TP7002")
 					(unit 1)
 				)
@@
 		(on_board yes)
 		(dnp no)
-		(property "Reference" "TP?"
+		(property "Reference" "TP7009"
 			(at 327.66 282.956 0)
 			(effects
@@
 			(project "v7_RK3588_PCB"
 				(path "/1d5a1342-f497-4807-8bdb-ea718133b0ad/fb1254ad-a22e-4d7b-81d8-e9d32dd5de93"
-					(reference "TP?")
+					(reference "TP7009")
 					(unit 1)
 				)
@@
 		(dnp no)
 		(fields_autoplaced yes)
-		(property "Reference" "TP?"
+		(property "Reference" "TP7011"
 			(at 414.02 324.3579 0)
 			(effects
@@
 			(project "v7_RK3588_PCB"
 				(path "/1d5a1342-f497-4807-8bdb-ea718133b0ad/fb1254ad-a22e-4d7b-81d8-e9d32dd5de93"
-					(reference "TP?")
+					(reference "TP7011")
 					(unit 1)
 				)
@@
 		(dnp no)
 		(fields_autoplaced yes)
-		(property "Reference" "Q?"
+		(property "Reference" "Q7004"
 			(at 360.68 275.5899 0)
 			(effects
@@
 			(project "v7_RK3588_PCB"
 				(path "/1d5a1342-f497-4807-8bdb-ea718133b0ad/fb1254ad-a22e-4d7b-81d8-e9d32dd5de93"
-					(reference "Q?")
+					(reference "Q7004")
 					(unit 1)
 				)
