File: v7_RK3588_PCB/WiFi.kicad_sch (KiCad schematic)
At the start: 0 parts

Commit message: add WiFi module
Parts:
- added 5001: *, symbol 453-00117_Sona IF573_SCH_Symbol_Altium:453-00117_Sona IF573_SCH_Symbol_Altium
Connections:
- new net GND: 5001.74 (GND), 5001.75 (GND), 5001.76 (GND), 5001.77 (GND), 5001.78 (GND), 5001.80 (GND), 5001.81 (GND), 5001.82 (GND), 5001.83 (GND), 5001.84 (GND), 5001.85 (GND), 5001.87 (GND)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
- no-connect marks 0 -> 3
