File: v7_RK3588_PCB/Power_Management.kicad_sch (KiCad schematic)
At the start: 107 parts, among them U3001 TPS62867RQYR, U3002 LTC4450AV-TRMPBF, U3003 TPS22811LRPWR, U3004 BQ27Z561YPHR-R2, U3005 TPS61088RHLR, U3006 LTC4450AV-TRMPBF, U3007 TPS22811LRPWR, U3008 SN74LVC1G32DBVR, U3010 LTC4450AV-TRMPBF, U3011 SN74LVC1G14DBVR, U3012 SN74LVC1G08DBVR, U3013 TPS2121RUXR, U3014 XTPS55285VALR, U3015 LTC4450AV-TRMPBF

Commit message: add 0ohm resistors on power management
Parts:
- added R3037, R3038, R3039, R3040, R3041, R3042, R3043, R3044, R3045: 0, symbol Device:R
Connections:
- net 5V0_OUT_ETH: now also R3037.1; no longer R3001.1, U3001.3 (VIN), U3001.4 (EN)
- net BATTERY_IN: now also R3041.1, R3042.2, R3043.2; no longer R3024.1, R3025.2, U3002.10 (OUT), U3002.11 (OUT), U3002.12 (OUT), U3002.13 (OUT), U3002.8 (OUT), U3002.9 (OUT), U3006.10 (OUT), U3006.11 (OUT), U3006.12 (OUT), U3006.13 (OUT), U3006.8 (OUT), U3006.9 (OUT)
- net BATTERY_PACK_OUT: now also R3040.2; no longer R3023.1, R3025.1
- net VCC3V3_SYS: now also R3038.2, R3039.2; no longer C3039.1, U3010.10 (OUT), U3010.11 (OUT), U3010.12 (OUT), U3010.13 (OUT), U3010.8 (OUT), U3010.9 (OUT), U3015.10 (OUT), U3015.11 (OUT), U3015.12 (OUT), U3015.13 (OUT), U3015.8 (OUT), U3015.9 (OUT)
- net at R3004.1, U3003.5 (IN): now also R3044.2; no longer BT3001.1 (+)
- net at R3015.1, U3007.5 (IN): now also R3045.2; no longer BT3002.1 (+)
- new net: R3023.1, R3025.1, R3040.1
- new net: R3043.1, U3006.10 (OUT), U3006.11 (OUT), U3006.12 (OUT), U3006.13 (OUT), U3006.8 (OUT), U3006.9 (OUT)
- new net: R3038.1, U3010.10 (OUT), U3010.11 (OUT), U3010.12 (OUT), U3010.13 (OUT), U3010.8 (OUT), U3010.9 (OUT)
- new net: R3024.1, R3025.2, R3041.2
- new net: BT3002.1 (+), R3045.1
- new net: BT3001.1 (+), R3044.1
- new net: R3042.1, U3002.10 (OUT), U3002.11 (OUT), U3002.12 (OUT), U3002.13 (OUT), U3002.8 (OUT), U3002.9 (OUT)
- new net: R3001.1, R3037.2, U3001.3 (VIN), U3001.4 (EN)
- new net: C3039.1, R3039.1, U3015.10 (OUT), U3015.11 (OUT), U3015.12 (OUT), U3015.13 (OUT), U3015.8 (OUT), U3015.9 (OUT)
Other:
- moved on the sheet: C3039
